Commit message: Automated update by GitHub Action

File: urdf/robot.urdf (robot description, URDF)
Before this commit: robot robot, 15 links, 14 joints
Links:
- removed link base_link
- added link imu_link, mass 1e-9
- added link motor_holder, mass 1.06123; collision mesh filename=package://catbot_leg_description/meshes/motor_holder.stl; collision mesh filename=package://catbot_leg_description/meshes/part_1.stl
- added link part_1, mass 1e-09; collision mesh filename=package://catbot_leg_description/meshes/part_1__3.stl; visual mesh filename=package://catbot_leg_description/meshes/part_1__3.stl
- added link part_1_2, mass 4.06535; collision mesh filename=package://catbot_leg_description/meshes/part_1__4.stl; visual mesh filename=package://catbot_leg_description/meshes/part_1__4.stl
Joints:
- added joint imu_link_frame: type fixed, parent motor_holder, child imu_link, origin xyz=0.6663 -0.0247675 0.518956 rpy=3.30424e-16 8.36432e-16 -2.58163e-15, axis 0 0 0
- added joint pitch: type revolute, parent part_1, child part_1_2, origin xyz=1.21116e-17 -0.149706 0.0105 rpy=-1.5708 1.5708 0, axis 0 0 1, limit lower=-3.141592653589793 upper=3.141592653589793 effort=10 velocity=10
- added joint yaw: type revolute, parent motor_holder, child part_1, origin xyz=1.11022e-16 0.0105 0.498956 rpy=1.5708 7.752e-16 -1.66569e-15, axis 0 0 1, limit lower=-3.141592653589793 upper=3.141592653589793 effort=10 velocity=10
- joint BR_leg1_1 (1) (1): origin xyz=-2.08167e-17 -6.93889e-18 0.029 rpy=3.14159 1.11382e-16 -1.20167 -> xyz=0 5.55112e-17 0.029 rpy=3.14159 1.11382e-16 -1.20167
- joint BR_leg_cyl_0_1 (1) (1): origin xyz=-2.08167e-17 -0.166278 0 rpy=3.14159 -2.45258e-33 -4.42072e-17 -> xyz=2.77556e-17 -0.166278 0 rpy=3.14159 3.7907e-32 1.13039e-17
- joint BR_leg_cyl_1_1 (1) (1): origin xyz=2.77556e-17 -0.207 0 rpy=3.14159 -3.97674e-31 5.83827e-17 -> xyz=2.77556e-17 -0.207 -1.11022e-16 rpy=-3.14159 -1.4511e-31 -6.07804e-18
- joint a: origin xyz=-0.005 -0.0645125 -0.0134017 rpy=1.5708 -1.25664 1.5708 -> xyz=0.6808 -0.0642675 0.432956 rpy=1.5708 -1.25664 1.5708; parent base_link -> motor_holder
- joint closing_BR_leg3_1 (1) (1)_1_frame: origin xyz=0.027272 -0.0419075 3.36536e-16 rpy=-3.0083e-16 2.4348e-15 -2.56468 -> xyz=0.027272 -0.0419075 2.22045e-16 rpy=-3.0083e-16 2.4348e-15 -2.56468
- joint closing_BR_leg3_1 (1) (1)_2_frame: origin xyz=-2.77556e-17 -0.207 0 rpy=3.14159 3.77607e-33 1.5708 -> xyz=0 -0.207 0 rpy=-3.14159 2.92432e-32 1.5708
- joint closing_BR_leg3_1 (1) (1)_2_z_frame: origin xyz=-2.77556e-17 -0.207 -0.1 rpy=3.14159 3.77607e-33 1.5708 -> xyz=2.77556e-17 -0.207 -0.1 rpy=-3.14159 2.92432e-32 1.5708
- joint l: origin xyz=-0.005 0.0645225 -0.0134017 rpy=-1.5708 0.628319 -1.5708 -> xyz=0.6808 0.0647675 0.432956 rpy=-1.5708 0.628319 -1.5708; parent base_link -> motor_holder

Commit message: Automated update by GitHub Action

File: urdf/robot.urdf (robot description, URDF)
Before this commit: robot robot, 18 links, 17 joints
Links:
- removed link base_link
- link imu_link: mass 1e-9 -> 1.06123; geometry collision mesh filename=package://catbot_leg_description/meshes/motor_holder.stl; collision mesh filename=package://catbot_leg_description/meshes/part_1.stl
- link part_1: geometry collision mesh filename=package://catbot_leg_description/meshes/part_1__4.stl; visual mesh filename=package://catbot_leg_description/meshes/part_1__4.stl
- link part_1_2: geometry collision mesh filename=package://catbot_leg_description/meshes/part_1__5.stl; visual mesh filename=package://catbot_leg_description/meshes/part_1__5.stl
Joints:
- removed joint imu_link_frame
- joint a: parent base_link -> imu_link
- joint l: parent base_link -> imu_link
- joint yaw: parent base_link -> imu_link

Commit message: Automated update by GitHub Action

File: urdf/robot.urdf (robot description, URDF)
Before this commit: robot robot, 17 links, 16 joints
Links:
- added link imu_link_motor_holder, mass 0.477236; collision mesh filename=package://catbot_leg_description/meshes/motor_holder.stl; visual mesh filename=package://catbot_leg_description/meshes/motor_holder.stl
- added link imu_link_part_1, mass 1e-09; collision mesh filename=package://catbot_leg_description/meshes/part_1.stl; visual mesh filename=package://catbot_leg_description/meshes/part_1.stl
- added link imu_link_part_1_2, mass 0.0319952; collision mesh filename=package://catbot_leg_description/meshes/part_1__2.stl; visual mesh filename=package://catbot_leg_description/meshes/part_1__2.stl
- added link imu_link_part_1_3, mass 0.26; collision mesh filename=package://catbot_leg_description/meshes/part_1__3.stl; visual mesh filename=package://catbot_leg_description/meshes/part_1__3.stl
- added link imu_link_part_1_4, mass 0.0319952; collision mesh filename=package://catbot_leg_description/meshes/part_1__2.stl; visual mesh filename=package://catbot_leg_description/meshes/part_1__2.stl
- added link imu_link_part_1_5, mass 0.26; collision mesh filename=package://catbot_leg_description/meshes/part_1__3.stl; visual mesh filename=package://catbot_leg_description/meshes/part_1__3.stl
- added link imu_link_t_slot_frame, mass 1e-09; collision mesh filename=package://catbot_leg_description/meshes/t_slot_frame.stl; visual mesh filename=package://catbot_leg_description/meshes/t_slot_frame.stl
- link imu_link: mass 1.06123 -> 1e-09; geometry 
Joints:
- added joint imu_link_motor_holder_fixed: type fixed, parent imu_link, child imu_link_motor_holder, origin xyz=0.6858 -0.0097675 0.450456 rpy=-3.14159 -3.30424e-16 1.5708, axis 0 0 1, limit effort=10 velocity=10
- added joint imu_link_part_1_2_fixed: type fixed, parent imu_link, child imu_link_part_1_2, origin xyz=0.6733 -0.0642675 0.432956 rpy=1.16838e-15 -1.91646e-16 1.5708, axis 0 0 1, limit effort=10 velocity=10
- added joint imu_link_part_1_3_fixed: type fixed, parent imu_link, child imu_link_part_1_3, origin xyz=0.6573 -0.0642675 0.432956 rpy=3.14159 0.464323 -1.5708, axis 0 0 1, limit effort=10 velocity=10
- added joint imu_link_part_1_4_fixed: type fixed, parent imu_link, child imu_link_part_1_4, origin xyz=0.6733 0.0647675 0.432956 rpy=1.16838e-15 -1.91646e-16 1.5708, axis 0 0 1, limit effort=10 velocity=10
- added joint imu_link_part_1_5_fixed: type fixed, parent imu_link, child imu_link_part_1_5, origin xyz=0.6573 0.0647675 0.432956 rpy=3.14159 0.464323 -1.5708, axis 0 0 1, limit effort=10 velocity=10
- added joint imu_link_part_1_fixed: type fixed, parent imu_link, child imu_link_part_1, origin xyz=0.654475 -0.00907667 0.518956 rpy=3.30424e-16 8.36432e-16 -2.58163e-15, axis 0 0 1, limit effort=10 velocity=10
- added joint imu_link_t_slot_frame_fixed: type fixed, parent imu_link, child imu_link_t_slot_frame, origin xyz=0.6958 0.0005 0.946156 rpy=-3.14159 -3.30424e-16 1.5708, axis 0 0 1, limit effort=10 velocity=10

Commit message: Automated update by GitHub Action

File: urdf/robot.urdf (robot description, URDF)
Before this commit: robot robot, 24 links, 23 joints
Links:
- removed link imu_link_motor_holder
- removed link imu_link_part_1
- removed link imu_link_part_1_2
- removed link imu_link_part_1_3
- removed link imu_link_part_1_4
- removed link imu_link_part_1_5
- removed link imu_link_t_slot_frame
- added link base_link, mass 1e-09
- added link base_link_motor_holder, mass 0.477236; collision mesh filename=package://catbot_leg_description/meshes/motor_holder.stl; visual mesh filename=package://catbot_leg_description/meshes/motor_holder.stl
- added link base_link_part_1, mass 0.0319952; collision mesh filename=package://catbot_leg_description/meshes/part_1.stl; visual mesh filename=package://catbot_leg_description/meshes/part_1.stl
- added link base_link_part_1_2, mass 0.26; collision mesh filename=package://catbot_leg_description/meshes/part_1__2.stl; visual mesh filename=package://catbot_leg_description/meshes/part_1__2.stl
- added link base_link_part_1_3, mass 0.0319952; collision mesh filename=package://catbot_leg_description/meshes/part_1.stl; visual mesh filename=package://catbot_leg_description/meshes/part_1.stl
- added link base_link_part_1_4, mass 0.26; collision mesh filename=package://catbot_leg_description/meshes/part_1__2.stl; visual mesh filename=package://catbot_leg_description/meshes/part_1__2.stl
- added link base_link_t_slot_frame, mass 1e-09; collision mesh filename=package://catbot_leg_description/meshes/t_slot_frame.stl; visual mesh filename=package://catbot_leg_description/meshes/t_slot_frame.stl
- link imu_link: mass 1e-09 -> 1e-9
- link part_1: geometry collision mesh filename=package://catbot_leg_description/meshes/part_1__3.stl; visual mesh filename=package://catbot_leg_description/meshes/part_1__3.stl
- link part_1_2: geometry collision mesh filename=package://catbot_leg_description/meshes/part_1__4.stl; visual mesh filename=package://catbot_leg_description/meshes/part_1__4.stl
Joints:
- removed joint imu_link_motor_holder_fixed
- removed joint imu_link_part_1_2_fixed
- removed joint imu_link_part_1_3_fixed
- removed joint imu_link_part_1_4_fixed
- removed joint imu_link_part_1_5_fixed
- removed joint imu_link_part_1_fixed
- removed joint imu_link_t_slot_frame_fixed
- added joint base_link_motor_holder_fixed: type fixed, parent base_link, child base_link_motor_holder, origin xyz=0.6858 -0.0097675 0.450456 rpy=-3.14159 -3.30424e-16 1.5708, axis 0 0 1, limit effort=10 velocity=10
- added joint base_link_part_1_2_fixed: type fixed, parent base_link, child base_link_part_1_2, origin xyz=0.6573 -0.0642675 0.432956 rpy=3.14159 0.464323 -1.5708, axis 0 0 1, limit effort=10 velocity=10
- added joint base_link_part_1_3_fixed: type fixed, parent base_link, child base_link_part_1_3, origin xyz=0.6733 0.0647675 0.432956 rpy=1.16838e-15 -1.91646e-16 1.5708, axis 0 0 1, limit effort=10 velocity=10
- added joint base_link_part_1_4_fixed: type fixed, parent base_link, child base_link_part_1_4, origin xyz=0.6573 0.0647675 0.432956 rpy=3.14159 0.464323 -1.5708, axis 0 0 1, limit effort=10 velocity=10
- added joint base_link_part_1_fixed: type fixed, parent base_link, child base_link_part_1, origin xyz=0.6733 -0.0642675 0.432956 rpy=1.16838e-15 -1.91646e-16 1.5708, axis 0 0 1, limit effort=10 velocity=10
- added joint base_link_t_slot_frame_fixed: type fixed, parent base_link, child base_link_t_slot_frame, origin xyz=0.6958 0.0005 0.946156 rpy=-3.14159 -3.30424e-16 1.5708, axis 0 0 1, limit effort=10 velocity=10
- added joint imu_link_frame: type fixed, parent base_link, child imu_link, origin xyz=0.6663 -0.0247675 0.518956 rpy=3.30424e-16 8.36432e-16 -2.58163e-15, axis 0 0 0
- joint a: parent imu_link -> base_link
- joint l: parent imu_link -> base_link
- joint yaw: parent imu_link -> base_link

Commit message: Automated update by GitHub Action

File: urdf/robot.urdf (robot description, URDF)
Before this commit: robot robot, 18 links, 17 joints
Joints:
- joint BR_leg1_1 (1) (1): origin xyz=-1.11022e-16 -1.66533e-16 0.029 rpy=-3.14159 5.73317e-16 -1.20167 -> xyz=-1.11022e-16 -1.11022e-16 0.029 rpy=-3.14159 6.91027e-16 -1.20167
- joint BR_leg2_1 (1) (1): origin xyz=0.0292942 0.0403199 0.029 rpy=-3.14159 1.34653e-15 -1.20023 -> xyz=0.0292942 0.0403199 0.029 rpy=3.14159 1.46668e-15 -1.20023
- joint BR_leg_cyl_0_1 (1) (1): origin xyz=2.77556e-17 -0.166278 -1.11022e-16 rpy=-3.14159 -6.74381e-32 -2.54852e-17 -> xyz=2.77556e-17 -0.166278 -1.11022e-16 rpy=-3.14159 -8.56299e-31 -2.54852e-17
- joint BR_leg_cyl_1_1 (1) (1): origin xyz=5.55112e-17 -0.207 -1.11022e-16 rpy=3.14159 -4.88264e-31 5.70903e-17 -> xyz=2.77556e-17 -0.207 -1.11022e-16 rpy=3.14159 -4.88264e-31 5.70903e-17
- joint l: limit lower=-0.174533 upper=2.18166 effort=10 velocity=10 -> lower=-1.0472 upper=2.18166 effort=10 velocity=10
